Commit message: x30 repaint

File: descriptions/deep_robotics/x30_description/xacro/body.xacro (robot description, xacro)
@@ -23,7 +23,6 @@
     <visual>
       <geometry>
-        <mesh filename="file://$(find x30_description)/meshes/torso.dae"/>
-      </geometry>
-      <material name="silver"/>
+        <mesh filename="file://$(find x30_description)/meshes/torso.obj"/>
+      </geometry>
     </visual>
     <collision>
@@ -42,7 +41,7 @@
     <visual>
       <geometry>
-        <mesh filename="file://$(find x30_description)/meshes/hip.dae"/>
-      </geometry>
-      <material name="grey"/>
+        <mesh filename="file://$(find x30_description)/meshes/fl_hip.STL"/>
+      </geometry>
+      <material name="silver"/>
     </visual>
   </link>
@@ -62,7 +61,6 @@
     <visual>
       <geometry>
-        <mesh filename="file://$(find x30_description)/meshes/l_thigh.dae"/>
-      </geometry>
-      <material name="light-grey"/>
+        <mesh filename="file://$(find x30_description)/meshes/l_thigh.obj"/>
+      </geometry>
     </visual>
     <collision>
@@ -88,5 +86,5 @@
     <visual>
       <geometry>
-        <mesh filename="file://$(find x30_description)/meshes/shank.dae"/>
+        <mesh filename="file://$(find x30_description)/meshes/shank.obj"/>
       </geometry>
       <material name="silver"/>
@@ -142,7 +140,7 @@
     <visual>
       <geometry>
-        <mesh filename="file://$(find x30_description)/meshes/hip.dae"/>
-      </geometry>
-      <material name="grey"/>
+        <mesh filename="file://$(find x30_description)/meshes/fr_hip.STL"/>
+      </geometry>
+      <material name="silver"/>
     </visual>
   </link>
@@ -162,7 +160,6 @@
     <visual>
       <geometry>
-        <mesh filename="file://$(find x30_description)/meshes/r_thigh.dae"/>
-      </geometry>
-      <material name="light-grey"/>
+        <mesh filename="file://$(find x30_description)/meshes/r_thigh.obj"/>
+      </geometry>
     </visual>
     <collision>
@@ -188,5 +185,5 @@
     <visual>
       <geometry>
-        <mesh filename="file://$(find x30_description)/meshes/shank.dae"/>
+        <mesh filename="file://$(find x30_description)/meshes/shank.obj"/>
       </geometry>
       <material name="silver"/>
@@ -242,7 +239,7 @@
     <visual>
       <geometry>
-        <mesh filename="file://$(find x30_description)/meshes/hip.dae"/>
-      </geometry>
-      <material name="grey"/>
+        <mesh filename="file://$(find x30_description)/meshes/hl_hip.STL"/>
+      </geometry>
+      <material name="silver"/>
     </visual>
   </link>
@@ -262,7 +259,6 @@
     <visual>
       <geometry>
-        <mesh filename="file://$(find x30_description)/meshes/l_thigh.dae"/>
-      </geometry>
-      <material name="light-grey"/>
+        <mesh filename="file://$(find x30_description)/meshes/l_thigh.obj"/>
+      </geometry>
     </visual>
     <collision>
@@ -288,5 +284,5 @@
     <visual>
       <geometry>
-        <mesh filename="file://$(find x30_description)/meshes/shank.dae"/>
+        <mesh filename="file://$(find x30_description)/meshes/shank.obj"/>
       </geometry>
       <material name="silver"/>
@@ -342,7 +338,7 @@
     <visual>
       <geometry>
-        <mesh filename="file://$(find x30_description)/meshes/hip.dae"/>
-      </geometry>
-      <material name="grey"/>
+        <mesh filename="file://$(find x30_description)/meshes/hr_hip.STL"/>
+      </geometry>
+      <material name="silver"/>
     </visual>
   </link>
@@ -362,7 +358,6 @@
     <visual>
       <geometry>
-        <mesh filename="file://$(find x30_description)/meshes/r_thigh.dae"/>
-      </geometry>
-      <material name="light-grey"/>
+        <mesh filename="file://$(find x30_description)/meshes/r_thigh.obj"/>
+      </geometry>
     </visual>
     <collision>
@@ -388,5 +383,5 @@
     <visual>
       <geometry>
-        <mesh filename="file://$(find x30_description)/meshes/shank.dae"/>
+        <mesh filename="file://$(find x30_description)/meshes/shank.obj"/>
       </geometry>
       <material name="silver"/>
