Commit message: feat: opt radio_link_input.py and go1 rviz.

File: descriptions/unitree/go1_description/xacro/depthCamera.xacro (robot description, xacro)
@@ -17,5 +17,5 @@
 				<origin xyz="0 0 0" rpy="0 0 0"/>
 				<geometry>
-					<mesh filename="file://$(find go1_description)/meshes/depthCamera.dae" scale="1 1 1"/>
+					<mesh filename="package://go1_description/meshes/depthCamera.dae" scale="1 1 1"/>
 				</geometry>
 			</visual>

File: descriptions/unitree/go1_description/xacro/leg.xacro (robot description, xacro)
@@ -60,5 +60,5 @@
         </xacro:if>
         <geometry>
-          <mesh filename="file://$(find go1_description)/meshes/hip.dae" scale="1 1 1"/>
+          <mesh filename="package://go1_description/meshes/hip.dae" scale="1 1 1"/>
         </geometry>
         <material name="deep-grey"/>
@@ -114,8 +114,8 @@
         <geometry>
           <xacro:if value="${mirror_dae == True}">
-            <mesh filename="file://$(find go1_description)/meshes/thigh.dae" scale="1 1 1"/>
+            <mesh filename="package://go1_description/meshes/thigh.dae" scale="1 1 1"/>
           </xacro:if>
           <xacro:if value="${mirror_dae == False}">
-            <mesh filename="file://$(find go1_description)/meshes/thigh_mirror.dae" scale="1 1 1"/>
+            <mesh filename="package://go1_description/meshes/thigh_mirror.dae" scale="1 1 1"/>
           </xacro:if>
         </geometry>
@@ -171,5 +171,5 @@
         <origin rpy="0 0 0" xyz="0 0 0"/>
         <geometry>
-          <mesh filename="file://$(find go1_description)/meshes/calf.dae" scale="1 1 1"/>
+          <mesh filename="package://go1_description/meshes/calf.dae" scale="1 1 1"/>
         </geometry>
         <material name="light-grey"/>

File: descriptions/unitree/go1_description/xacro/robot.xacro (robot description, xacro)
@@ -49,5 +49,5 @@
 			<origin rpy="0 0 0" xyz="0 0 0"/>
 			<geometry>
-				<mesh filename="file://$(find go1_description)/meshes/trunk.dae" scale="1 1 1"/>
+				<mesh filename="package://go1_description/meshes/trunk.dae" scale="1 1 1"/>
 			</geometry>
 			<material name="light-grey"/>

File: descriptions/unitree/go1_description/xacro/ultraSound.xacro (robot description, xacro)
@@ -17,5 +17,5 @@
 				<origin xyz="0 0 0" rpy="0 0 0"/>
 				<geometry>
-					<mesh filename="file://$(find go1_description)/meshes/ultraSound.dae" scale="1 1 1"/>
+					<mesh filename="package://go1_description/meshes/ultraSound.dae" scale="1 1 1"/>
 				</geometry>
 				<material name="black"/>
